Commit message: update body and urdf

File: model/sample_robot_description/urdf/sample_robot_reduced.urdf (robot description, URDF)
Before this commit: robot sample_robot, 36 links, 35 joints
Joints:
- joint L_LOWERARM_P: origin xyz=0.0 -8.32667268469e-17 -0.2 rpy=0.0 -1.0 0.0 -> xyz=0.0 -8.32667268469e-17 -0.2 rpy=0.0 0.0 0.0
- joint L_UPPERARM_P: origin xyz=0.0 0.1 0.1 rpy=0.3 0.5 0.0 -> xyz=0.0 0.1 0.1 rpy=0.0 0.0 0.0
- joint R_LOWERARM_P: origin xyz=0.0 0.0 -0.2 rpy=0.0 -1.0 0.0 -> xyz=0.0 0.0 -0.2 rpy=0.0 0.0 0.0
- joint R_UPPERARM_P: origin xyz=0.0 -0.1 0.1 rpy=-0.3 0.5 0.0 -> xyz=0.0 -0.1 0.1 rpy=0.0 0.0 0.0
